File: Driver-Board.kicad_pcb (KiCad board)
At the start: 2 copper layers, 5 parts, among them IC1 ATTINY45-S, P1 CONN_4

Commit message: Added some stuff to the 'Driver-Board'.
Parts:
- removed R17: R, MADW__R0805
- added R1: 10k, MADW__R0805, F.Cu at (135.6, 91.9)
- added R2: 15, MADW__R0805, F.Cu at (135.9, 103.2)
- added R3: 15, MADW__R0805, F.Cu at (132.9, 97.7)
Connections:
- IC1 pad 2: (no net) -> N-000004
- IC1 pad 3: (no net) -> N-000003
- P1 pad 2: (no net) -> /sink
- P1 pad 3: (no net) -> VCC
