File: Driver-Board.sch (KiCad schematic (older format))
At the start: 5 parts, among them IC1 ATTINY45-S, P1 CONN_4

Commit message: Added some stuff to the 'Driver-Board'.
Parts:
- added R2, R3: 15, symbol R
- R1: renamed from R17; value R -> 10k
Connections:
- net VCC: now also P1.3 (P3)
- net sink: now reaches P1.2 (P2)
- net sink: now also R2.1, R3.1
- net at IC1.2 (PB3(XTAL1/CLKI/OC1B/ADC3/PCINT3)): now also R2.2
- net at IC1.3 (PB4(XTAL2/CLKO/OC1B/ADC2/PCINT4)): now also R3.2
- no-connect marks 4 -> 0
Changed lines of the file:
@@
 Text GLabel 3350 2900 0    39   Input ~ 0
 SCK
-NoConn ~ 3450 3000
-NoConn ~ 3450 3100
 Wire Wire Line
 	4950 1700 5200 1700
@@
 	3350 2900 3450 2900
 $Comp
-L R R17
+L R R1
 U 1 1 5234931E
 P 3350 3450
-F 0 "R17" V 3430 3450 40  0000 C CNN
-F 1 "R" V 3357 3451 40  0000 C CNN
+F 0 "R1" V 3430 3450 40  0000 C CNN
+F 1 "10k" V 3357 3451 40  0000 C CNN
 F 2 "" V 3280 3450 30  0000 C CNN
 F 3 "" H 3350 3450 30  0000 C CNN
@@
 	1    0    0    -1
 $EndComp
+Wire Wire Line
+	5000 2000 5000 2100
+Wire Wire Line
+	5000 1600 5000 1800
+$Comp
+L ATTINY45-S IC1
+U 1 1 52348D75
+P 4800 2950
+F 0 "IC1" H 3650 3350 40  0000 C CNN
+F 1 "ATTINY45-S" H 5800 2550 40  0000 C CNN
+F 2 "SO8-200" H 5750 2950 35  0000 C CIN
+F 3 "" H 4800 2950 60  0000 C CNN
+	1    4800 2950
+	1    0    0    -1
+$EndComp
+Wire Wire Line
+	5000 1800 4950 1800
+$Comp
+L R R2
+U 1 1 5234962E
+P 2900 3000
+F 0 "R2" V 3000 3000 40  0000 C CNN
+F 1 "15" V 2900 3000 40  0000 C CNN
+F 2 "" V 2830 3000 30  0000 C CNN
+F 3 "" H 2900 3000 30  0000 C CNN
+	1    2900 3000
+	0    -1   -1   0
+$EndComp
+$Comp
+L R R3
+U 1 1 52349642
+P 2900 3100
+F 0 "R3" V 2800 3100 40  0000 C CNN
+F 1 "15" V 2907 3101 40  0000 C CNN
+F 2 "" V 2830 3100 30  0000 C CNN
+F 3 "" H 2900 3100 30  0000 C CNN
+	1    2900 3100
+	0    -1   -1   0
+$EndComp
+Wire Wire Line
+	3150 3000 3450 3000
+Wire Wire Line
+	3450 3100 3150 3100
+Wire Wire Line
+	2650 3000 2600 3000
+Wire Wire Line
+	2600 3000 2600 3100
+Wire Wire Line
+	2600 3100 2650 3100
+Text Label 2550 3050 2    60   ~ 0
+sink
+Wire Wire Line
+	2550 3050 2600 3050
+Connection ~ 2600 3050
 $Comp
 L CONN_4 P1
@@
 	-1   0    0    1
 $EndComp
-NoConn ~ 4950 1800
-NoConn ~ 4950 1900
+Text Label 5000 1900 0    60   ~ 0
+sink
 Wire Wire Line
-	5000 2000 5000 2100
-Wire Wire Line
-	5000 1700 5000 1600
-$Comp
-L ATTINY45-S IC1
-U 1 1 52348D75
-P 4800 2950
-F 0 "IC1" H 3650 3350 40  0000 C CNN
-F 1 "ATTINY45-S" H 5800 2550 40  0000 C CNN
-F 2 "SO8-200" H 5750 2950 35  0000 C CIN
-F 3 "" H 4800 2950 60  0000 C CNN
-	1    4800 2950
-	1    0    0    -1
-$EndComp
+	4950 1900 5000 1900
 $EndSCHEMATC
